Commit message: feat: Enable Gazebo hardware acceleration, refine random walker logic, and update TurtleBot3 URDF to a standard format.

File: src/robot_gazebo_sim/urdf/turtlebot3_burger.urdf (robot description, URDF)
Before this commit: robot turtlebot3_burger, 9 links, 8 joints
Links:
- removed link ${namespace}base_footprint
- removed link ${namespace}base_link
- removed link ${namespace}base_scan
- removed link ${namespace}camera_link
- removed link ${namespace}camera_optical_frame
- removed link ${namespace}caster_back_link
- removed link ${namespace}imu_link
- removed link ${namespace}wheel_left_link
- removed link ${namespace}wheel_right_link
- added link base_footprint
- added link base_link, mass 8.2573504e-01; collision box size=0.140 0.140 0.143; visual mesh filename=package://turtlebot3_descriptions/meshes/bases/burger_base.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 scale=0.001 0.001 0.001
- added link base_scan, mass 0.114; collision cylinder length=0.0315 radius=0.055; visual mesh filename=package://turtlebot3_descriptions/meshes/sensors/lds.stl scale=0.001 0.001 0.001
- added link caster_back_link, mass 0.005; collision box size=0.030 0.009 0.020
- added link imu_link
- added link oak_d_pro_camera, mass 0.09100000; collision box size=0.1 0.03 0.02; visual box size=0.1 0.03 0.02
- added link oak_d_pro_color_optical_frame
- added link oak_d_pro_depth_optical_frame
- added link wheel_left_link, mass 2.8498940e-02; collision cylinder length=0.018 radius=0.033; visual mesh filename=package://turtlebot3_descriptions/meshes/wheels/left_tire.s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 scale=0.001 0.001 0.001
- added link wheel_right_link, mass 2.8498940e-02; collision cylinder length=0.018 radius=0.033; visual mesh filename=package://turtlebot3_descriptions/meshes/wheels/right_tire.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 scale=0.001 0.001 0.001
Joints:
- removed joint ${namespace}base_joint
- removed joint ${namespace}camera_joint
- removed joint ${namespace}camera_optical_joint
- removed joint ${namespace}caster_back_joint
- removed joint ${namespace}imu_joint
- removed joint ${namespace}scan_joint
- removed joint ${namespace}wheel_left_joint
- removed joint ${namespace}wheel_right_joint
- added joint base_joint: type fixed, parent base_footprint, child base_link, origin xyz=0.0 0.0 0.010 rpy=0 0 0
- added joint caster_back_joint: type fixed, parent base_link, child caster_back_link, origin xyz=-0.081 0 -0.004 rpy=-1.57 0 0
- added joint imu_joint: type fixed, parent base_link, child imu_link, origin xyz=-0.032 0 0.068 rpy=0 0 0
- added joint joint_oak_d_pro_camera: type fixed, parent base_link, child oak_d_pro_camera, origin xyz=0.065 0.0 0.11 rpy=1.57 0.0 1.57
- added joint joint_oak_d_pro_color_optical_frame: type fixed, parent oak_d_pro_camera, child oak_d_pro_color_optical_frame, origin xyz=0.0 0.0 0.0 rpy=-1.5708 0.0 -1.5708
- added joint oak_d_pro_depth_optical_frame: type fixed, parent oak_d_pro_camera, child oak_d_pro_depth_optical_frame, origin xyz=0.0 0.0 0.0 rpy=-1.5708 0.0 -1.5708
- added joint scan_joint: type fixed, parent base_link, child base_scan, origin xyz=-0.032 0 0.172 rpy=0 0 0
- added joint wheel_left_joint: type continuous, parent base_link, child wheel_left_link, origin xyz=0.0 0.08 0.023 rpy=-1.57 0 0, axis 0 0 1
- added joint wheel_right_joint: type continuous, parent base_link, child wheel_right_link, origin xyz=0.0 -0.080 0.023 rpy=-1.57 0 0, axis 0 0 1

Commit message: fix: Update OAK-D-PRO camera box dimensions and joint rotation in URDF.

File: src/robot_gazebo_sim/urdf/turtlebot3_burger.urdf (robot description, URDF)
Before this commit: robot turtlebot3_burger, 10 links, 9 joints
Joints:
- joint joint_oak_d_pro_camera: origin xyz=0.065 0.0 0.11 rpy=1.57 0.0 1.57 -> xyz=0.065 0.0 0.11 rpy=0.0 0.0 0.0
