Commit message: Implémentation fonctionnelle avec camera OAK_D et CATAPAF

File: src/catapaf_gazebo/urdf/turtlebot_catapaf.urdf (robot description, URDF)
Before this commit: robot turtlebot3_burger_cam1, 11 links, 10 joints
Links:
- removed link camera_link
- removed link camera_rgb_frame
- removed link camera_rgb_optical_frame
- added link catapaf_arm, mass 0.05000000; collision box size=0.12 0.05 0.03; visual mesh filename=package://catapaf_gazebo/models/catapaf_common/meshes/catap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
- added link catapaf_base, mass 0.15; collision box size=0.08 0.05 0.03; visual mesh filename=package://catapaf_gazebo/models/catapaf_common/meshes/catap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
- added link oak_d_pro_camera, mass 0.091; collision box size=0.1 0.03 0.02; visual mesh filename=package://catapaf_gazebo/models/catapaf_common/meshes/senso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
- added link oak_d_pro_color_optical_frame
- added link oak_d_pro_depth_optical_frame
Joints:
- removed joint camera_joint
- removed joint camera_rgb_joint
- removed joint camera_rgb_optical_joint
- added joint catapaf_base_mount: type fixed, parent base_link, child catapaf_base, origin xyz=-0.03 -0.09 0.11
- added joint catapaf_joint: type revolute, parent catapaf_base, child catapaf_arm, origin xyz=0 -0.008 0 rpy=3.14159265359 3.14159265359 0, axis 0 1 0, limit lower=-1.5 upper=1.3 effort=1.0 velocity=5.0
- added joint joint_oak_d_pro_camera: type fixed, parent base_link, child oak_d_pro_camera, origin xyz=0.065 0 0.11 rpy=0 0 0
- added joint joint_oak_d_pro_color_optical_frame: type fixed, parent oak_d_pro_camera, child oak_d_pro_color_optical_frame, origin xyz=0 0 0 rpy=-1.5707 0 -1.5707
- added joint joint_oak_d_pro_depth_optical_frame: type fixed, parent oak_d_pro_camera, child oak_d_pro_depth_optical_frame, origin xyz=0 0 0 rpy=-1.5707 0 -1.5707
- joint camera_depth_joint: parent camera_link -> oak_d_pro_camera

Commit message: refacto urdf et sdf  hotfix setup.py

File: src/catapaf_gazebo/urdf/turtlebot_catapaf.urdf (robot description, URDF)
Before this commit: robot turtlebot3_burger_cam1, 13 links, 12 joints
Links:
- removed link camera_depth_optical_frame
Joints:
- removed joint camera_depth_joint

Commit message: Robot fonctionnel avec ball spawner et controller (il a la tremblote)

File: src/catapaf_gazebo/urdf/turtlebot_catapaf.urdf (robot description, URDF)
Before this commit: robot turtlebot3_burger_cam1, 12 links, 11 joints
Links:
- link catapaf_arm: geometry collision mesh filename=package://catapaf_gazebo/models/catapaf_common/meshes/catap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; visual mesh filename=package://catapaf_gazebo/models/catapaf_common/meshes/catap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
