Commit message: Simplification du controller du bras et patch des inerties

File: src/catapaf_gazebo/urdf/turtlebot_catapaf_simple.urdf (robot description, URDF)
Before this commit: robot turtlebot3_burger_cam1, 14 links, 13 joints
Joints:
- joint catapaf_joint: limit lower=-1.5 upper=0 effort=20.0 velocity=200.0 -> lower=-1.5 upper=0.2 effort=1.0 velocity=5.0
